Commit message: fixes to get this to work under ros humble

File: omni_description/urdf/omni.xacro (robot description, xacro)
@@ -1,4 +1,5 @@
 <?xml version="1.0" encoding="utf-8"?>
-<robot name="phantom_omni" xmlns:xacro="http://www.ros.org/wiki/xacro">
+<robot xmlns:xacro="http://www.ros.org/wiki/xacro">
+  <xacro:macro name="omni">
 	<!-- Materials -->
 	<material name="metal_seamed">
@@ -119,3 +120,4 @@
     <limit lower="-2.58" upper="2.58" velocity="100" effort="5" />
   </joint>
+  </xacro:macro>
 </robot>
